Commit message: Remove unused properties

File: urdf/turtlebot3_monster.urdf.xacro (robot description, xacro)
@@ -5,8 +5,4 @@
   <!-- <xacro:include filename="$(find realsense2_camera)/urdf/_d435.urdf.xacro"/> -->
   <xacro:include filename="$(find zed_wrapper)/urdf/zedm.urdf"/>
-  <xacro:property name="r200_cam_rgb_px" value="0.005"/>
-  <xacro:property name="r200_cam_rgb_py" value="0.018"/>
-  <xacro:property name="r200_cam_rgb_pz" value="0.013"/>
-  <xacro:property name="r200_cam_depth_offset" value="0.01"/>
   <link name="base_footprint"/>
   <joint name="base_joint" type="fixed">

Commit message: Avoid name clash in imu_link from TB3 and ZEDM

File: urdf/turtlebot3_monster.urdf.xacro (robot description, xacro)
@@ -4,5 +4,4 @@
   <xacro:include filename="$(find turtlebot3_description)/urdf/turtlebot3_waffle.gazebo.xacro"/>
   <!-- <xacro:include filename="$(find realsense2_camera)/urdf/_d435.urdf.xacro"/> -->
-  <xacro:include filename="$(find zed_wrapper)/urdf/zedm.urdf"/>
   <link name="base_footprint"/>
   <joint name="base_joint" type="fixed">
@@ -134,5 +133,5 @@
     <origin xyz="0.0 0 0.068" rpy="0 0 0"/>
   </joint>
-  <!-- <link name="imu_link"/> -->
+  <link name="imu_link"/>
   <joint name="scan_joint" type="fixed">
     <parent link="base_link"/>
@@ -162,9 +161,21 @@
     </inertial>
   </link>
+  <!-- ZEDM -->
+  <link name="zed_camera_link">
+    <visual>
+      <geometry>
+        <mesh filename="package://zed_wrapper/urdf/ZEDM.stl" />
+      </geometry>
+      <material name="light_grey">
+        <color rgba="0 0 0 0.9"/>
+      </material>
+    </visual>
+  </link>
   <joint name="zed_camera_joint" type="fixed">
     <origin xyz="0.031 -0.008163 0.151843" rpy="0 0 0"/>
     <parent link="base_link"/>
-    <child link="zed_camera_center"/>
+    <child link="zed_camera_link"/>
   </joint>
+  <!-- REALSENSE D435 -->
   <!-- <sensor_d435 parent="base_link"> -->
   <!--   <origin xyz="0.049 0.0 0.1795" rpy="0 0 0"/> -->

Commit message: Add realsense D435 bringup

File: urdf/turtlebot3_monster.urdf.xacro (robot description, xacro)
@@ -3,5 +3,5 @@
   <xacro:include filename="$(find turtlebot3_description)/urdf/common_properties.xacro"/>
   <xacro:include filename="$(find turtlebot3_description)/urdf/turtlebot3_waffle.gazebo.xacro"/>
-  <!-- <xacro:include filename="$(find realsense2_camera)/urdf/_d435.urdf.xacro"/> -->
+  <xacro:include filename="$(find realsense2_camera)/urdf/_d435.urdf.xacro"/>
   <link name="base_footprint"/>
   <joint name="base_joint" type="fixed">
@@ -178,6 +178,6 @@
   </joint>
   <!-- REALSENSE D435 -->
-  <!-- <sensor_d435 parent="base_link"> -->
-  <!--   <origin xyz="0.049 0.0 0.1795" rpy="0 0 0"/> -->
-  <!-- </sensor_d435> -->
+  <sensor_d435 parent="base_link">
+    <origin xyz="0.049 0.0 0.1795" rpy="0 0 0"/>
+  </sensor_d435>
 </robot>
