Commit message: Update zedm and d435 description files

File: urdf/waffle_deep.urdf.xacro (robot description, xacro)
@@ -3,5 +3,5 @@
   <xacro:include filename="$(find turtlebot3_description)/urdf/common_properties.xacro"/>
   <xacro:include filename="$(find turtlebot3_description)/urdf/turtlebot3_waffle.gazebo.xacro"/>
-  <xacro:include filename="$(find realsense2_camera)/urdf/_d435.urdf.xacro"/>
+  <xacro:include filename="$(find realsense2_description)/urdf/_d435.urdf.xacro"/>
   <link name="base_footprint"/>
   <joint name="base_joint" type="fixed">
@@ -165,5 +165,5 @@
     <visual>
       <geometry>
-        <mesh filename="package://zed_wrapper/urdf/ZEDM.stl" />
+        <mesh filename="package://turtlebot3_slam_3d/urdf/ZEDM.stl" />
       </geometry>
       <material name="light_grey">
